File: hardware/eprintedexam.sch (KiCad schematic (older format))
At the start: 49 parts, among them J1 Conn_01x04, J2 Conn_01x08, Q1 2N7002, Q2 2N7002, Q3 2N7002, Q4 2N7002, Q5 2N7002, Q6 2N7002, SW1 SW_Push, SW2 SW_Push, SW3 SW_Push, SW4 SW_Push, U1 AP1117-33, U2 ESP-12F

Commit message: mayor hardware change, fixed bad mosfet connection, increase c6 value to 37uF and decreased R1 to 1k and R10 to 3.3k, and tidy up the pcb desing so fast traces are length minimized
Parts:
- removed C1, C5, C7: 100n, Capacitor_SMD:C_1206_3216Metric, symbol Device:C
- removed R11: 33k, Resistor_SMD:R_1206_3216Metric, symbol Device:R
- removed R16: 10k, Resistor_SMD:R_1206_3216Metric, symbol Device:R
- removed R6, R7: 1k, Resistor_SMD:R_1206_3216Metric, symbol Device:R
- added C1: 100u, Capacitor_THT:CP_Radial_D8.0mm_P5.00mm, symbol Device:CP1
- added C2: 220u, Capacitor_THT:CP_Radial_D10.0mm_P5.00mm, symbol Device:CP1
- added C6: 47u, Capacitor_THT:CP_Radial_D6.3mm_P2.50mm, symbol Device:CP1
- added D1: 2N7001, Diode_THT:D_DO-35_SOD27_P10.16mm_Horizontal, symbol Device:D
- added R2: 33k, Resistor_SMD:R_1206_3216Metric, symbol Device:R
- C7: renamed from C6; value 10n -> 100n
- D2: renamed from D1; value D -> 2N7001
- R1: renamed from R12; value 10k -> 1k
- R10: renamed from R14; value 22k -> 3.3k
- R13: renamed from R17; value 560k -> 680k
- renumbered C2 to C3, C3 to C4, C4 to C5, R15 to R11, R18 to R12, R2 to R3, R3 to R4, R4 to R5, R8 to R6, R9 to R7, R10 to R8, R13 to R9
Connections:
- net GND: now also Q4.2 (S), C1.2, C2.2, R2.2; no longer Q4.3 (D), U1.1 (GND)
- net VCC: now also R12.1, C2.1, D1.2 (A), R2.1; no longer R12.2
- net nrst: now also Q4.3 (D), C6.1; no longer Q4.2 (S)
- net nxt: now also SW3.2
- net nxt+prv: now also C6.2
- net prv: now also SW4.2
- net spi-nrst: now also R12.2; no longer R12.1
- net spi-rst: now also Q6.1 (G)
- net at BT1.1 (+), U1.3 (VI): now also D1.1 (K)
- new net: C1.1, U1.1 (GND)
Other:
- note added: "gpio2 pullup in OR gate component"
- note added: "logic OR of singals prv and nxt"
- note added: "not gate for spi-rst signal"
- note removed: "gpio2 pullup in NOR gate component"
- note removed: "logic NOR of singals prv and nxt"
- note removed: "not gate for spi-rst singal"
- note removed: "nrts pullup in monostable component"
- moved on the sheet: BT1, D2, Q4, Q6, R1, R11, R12, SW1, SW3, SW4, U1
