File: hardware/_autosave-eprintedexam.kicad_pcb (KiCad board)
At the start: 2 copper layers, 103 x 98.5 mm, 57 parts, among them J1 Conn_01x04, J2 Conn_01x08, Q1 2N7002, Q2 2N7002, Q3 2N7002, Q4 2N7002, Q5 2N7002, Q6 2N7002, Q7 2N7002, Q8 2N7002, Q9 2N7002, SW1 SW_Push, SW2 SW_Push, SW3 SW_Push, SW4 SW_Push, U1 AP1117-33, U2 ESP-12F

Commit message: the hardware works
Parts:
- added R10: 33k, Resistor_SMD:R_1206_3216Metric, F.Cu at (75.4, 64.6)
- C3: renamed from C1; footprint Capacitor_THT:CP_Radial_D8.0mm_P5.00mm -> Capacitor_THT:CP_Radial_D6.3mm_P2.50mm
- C4: renamed from C2; footprint Capacitor_THT:CP_Radial_D10.0mm_P5.00mm -> Capacitor_THT:CP_Radial_D6.3mm_P2.50mm
- R14: renamed from R20; value 1k -> 10k
- moved R7 7.36 mm to (61.4, 63.3)
- moved TP6 5.56 mm to (72.6, 58.2)
- moved C4 2.37 mm to (118.2, 61.3), turned to 180 degrees
- moved SW3 2.34 mm to (76.8, 58.6), turned to 270 degrees
- moved D1 1.07 mm to (121.5, 38.6)
- moved C3 0.26 mm to (110.8, 61.3)
- renumbered C4 to C1, C5 to C2, C6 to C5, C7 to C6, C3 to C7, J2 to J1, J1 to J2, Q3 to Q1, Q4 to Q2, Q5 to Q3, Q6 to Q4, Q7 to Q5, Q8 to Q6, Q9 to Q7, Q1 to Q8, Q2 to Q9, R9 to R1, R18 to R11, R14 to R12, R19 to R13, R3 to R15, R7 to R16, R8 to R17, R10 to R18, R11 to R19, R12 to R2, R13 to R3, R2 to R4, R15 to R5, R4 to R6, R6 to R7, R16 to R8, R17 to R9, SW3 to SW1, SW4 to SW2, SW2 to SW3, SW1 to SW4
Routing:
- net spi-rst: track 85.6 -> 109.5 mm
- net VCC: track 240.9 -> 249.5 mm
- net GND: track 20.1 -> 17.3 mm
- net spi-busy,flash: track 84.2 -> 85.2 mm
- net Net-(BT1-Pad1): track 47.4 -> 46.8 mm
